File: Lion-Schutz.kicad_sch (KiCad schematic)
At the start: 29 parts, among them J1 USB_C, Q1 BSS806N, Q2 BSS806N, U1 TPS631000, U5 DW01A, U6 TP4056-42-ESOP8

Commit message: Added README
Other:
- title: (none) -> Lion Schutz PCB
Changed lines of the file:
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@@
 	(generator_version "10.0")
 	(paper "A4")
+	(title_block
+		(title "Lion Schutz PCB")
+		(date "2026-03-29")
+		(rev "0.1")
+	)
 	(text "USB"
 		(exclude_from_sim no)
